Commit message: aligned urdf with arm calibration zero position, added joint limits

File: URDF/SO_5DOF_ARM100_8j_URDF.SLDASM/urdf/SO_5DOF_ARM100_8j_URDF.SLDASM.urdf (robot description, URDF)
Before this commit: robot SO_5DOF_ARM100_8j_URDF.SLDASM, 7 links, 6 joints
Links:
- added link Root
- link Base: geometry collision mesh filename=../meshes/Base.STL; visual mesh filename=../meshes/Base.STL
- link Fixed_Jaw: geometry collision mesh filename=../meshes/Fixed_Jaw.STL; visual mesh filename=../meshes/Fixed_Jaw.STL
- link Lower_Arm: geometry collision mesh filename=../meshes/Lower_Arm.STL; visual mesh filename=../meshes/Lower_Arm.STL
- link Moving Jaw: geometry collision mesh filename=../meshes/Moving Jaw.STL; visual mesh filename=../meshes/Moving Jaw.STL
- link Rotation_Pitch: geometry collision mesh filename=../meshes/Rotation_Pitch.STL; visual mesh filename=../meshes/Rotation_Pitch.STL
- link Upper_Arm: geometry collision mesh filename=../meshes/Upper_Arm.STL; visual mesh filename=../meshes/Upper_Arm.STL
- link Wrist_Pitch_Roll: geometry collision mesh filename=../meshes/Wrist_Pitch_Roll.STL; visual mesh filename=../meshes/Wrist_Pitch_Roll.STL
Joints:
- added joint fixed_joint: type fixed, parent Root, child Base, origin xyz=0 0 0 rpy=0 0 1.5708
- joint Elbow: limit (none) -> lower=0 upper=3.14 effort=200.0 velocity=2; origin xyz=0 0.11257 0.028 rpy=0 0 0 -> xyz=0 0.11257 0.028 rpy=-1.5708 0 0
- joint Jaw: limit (none) -> lower=0 upper=1.57 effort=200.0 velocity=2
- joint Pitch: axis 1 0 0 -> -1 0 0; limit (none) -> lower=0 upper=3.4 effort=200.0 velocity=2; origin xyz=0 0.1025 0.0306 rpy=0 0 0 -> xyz=0 0.1025 0.0306 rpy=1.5708 0 0
- joint Rotation: limit (none) -> lower=-1.57 upper=1.57 effort=200.0 velocity=2
- joint Wrist_Pitch: limit (none) -> lower=-1.57 upper=1.57 effort=200.0 velocity=2; origin xyz=0 0.0052 0.1349 rpy=0 0 0 -> xyz=0 0.0052 0.1349 rpy=-1.5708 0 0
- joint Wrist_Roll: limit (none) -> lower=-2.5 upper=2.5 effort=200.0 velocity=2; origin xyz=0 -0.0601 0 rpy=0 0 0 -> xyz=0 -0.0601 0 rpy=0 1.5708 0

Commit message: changes axes which differed on real robot

File: URDF/SO_5DOF_ARM100_8j_URDF.SLDASM/urdf/SO_5DOF_ARM100_8j_URDF.SLDASM.urdf (robot description, URDF)
Before this commit: robot SO_5DOF_ARM100_8j_URDF.SLDASM, 8 links, 7 joints
Joints:
- joint Rotation: axis 0 1 0 -> 0 -1 0
- joint Wrist_Roll: axis 0 1 0 -> 0 -1 0
